File: hardware/cube-cover.kicad_pcb (KiCad board)
At the start: 2 copper layers, 120 x 120 mm, 16 parts

Commit message: Replace Order_Number
Parts:
- H101, H102, H103, H104: value Mounting_Hole -> 2mm_Pad_4mm
- H105: value MountingHole_1mm -> 1mm
- H106, H107, H110, H111: value Mounting_Hole -> 3mm_Pad_8mm
- INFO101: value ORDER-NUMBER -> ~; footprint V2_Production:Order_Number -> V2_Production:Revision

Commit message: Update Library
Parts:
- renumbered SWT102 to CON102, SWT103 to CON103
Changed lines of the file:
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@@
 		(layer "F.Cu")
 		(at 190 96.25)
-		(property "Reference" "SWT103"
+		(property "Reference" "CON103"
 			(at 0 -13.8 0)
 			(layer "F.SilkS")
@@
 		)
 		(group ""
-			(members "4d28e2c4-4ad8-4979-bf4d-34e8b7c7474a" "73266999-807a-4fa0-8454-0f49fc6c8ee7"
-				"b2a497b3-51f5-45cd-9d46-f165ad49594d" "b320016c-aecb-4f42-80ec-7a2514e6e566"
-				"b4dbae29-8f2b-459e-982b-58310bce9b49"
+			(members "2676dc9b-fcb6-4507-acc9-cd5cdd492143" "3fbcc421-3bc9-4848-abad-2aa953e0de26"
+				"56664212-955b-4178-9f0b-b3c6300e0f1f" "689f38a3-8174-45ac-b1ee-5a22d8b99268"
+				"eee2cbb3-98f7-4266-ab87-5ea827ec0d0f"
 			)
 		)
 		(group ""
-			(members "0d7c65df-4cd8-4635-8cc3-b7960ad28ea4" "4da047ac-e7e5-4171-9000-52704af13cd1"
-				"5336ec61-6e7a-48a4-af59-ee7ac7b0b2c4" "5c74deab-8f9b-413f-9476-54930fb8ff8b"
-				"726d6fbc-1b14-48c3-b043-96a848f9c79a"
+			(members "78e48961-dca4-42ba-9ccd-049f5865e259" "a8203589-7add-4c07-847b-0c8b89b5c8ca"
+				"ad2cc218-429d-483d-a516-472b1b260768" "cc454cb2-9a6d-4b4e-b11e-a0c9f761a3ae"
+				"de931184-a008-42fb-819e-63698c51ef79"
 			)
 		)
@@
 		(layer "F.Cu")
 		(at 164 96.25)
-		(property "Reference" "SWT102"
+		(property "Reference" "CON102"
 			(at 0 -13.8 0)
 			(layer "F.SilkS")
